Commit message: edit urdf and xml

File: data/a1/urdf/a1.urdf (robot description, URDF)
Before this commit: robot a1_description, 19 links, 18 joints
Joints:
- removed joint floating_base
- added joint : type floating, parent world, child trunk, origin xyz=0 0 0 rpy=0 0 0

File: data/aliengo/urdf/aliengo.urdf (robot description, URDF)
Before this commit: robot aliengo_description, 19 links, 18 joints
Joints:
- removed joint floating_base
- added joint : type floating, parent world, child trunk, origin xyz=0 0 0 rpy=0 0 0

File: data/laikago/urdf/laikago.urdf (robot description, URDF)
Before this commit: robot laikago_description, 14 links, 13 joints
Joints:
- removed joint floating_base
- added joint : type floating, parent world, child trunk, origin xyz=0 0 0 rpy=0 0 0
