Commit message: edit xml and python script

File: data/aliengo/urdf/aliengo.urdf (robot description, URDF)
Before this commit: robot aliengo_description, 19 links, 18 joints
Links:
- removed link base
- added link world
Joints:
- joint floating_base: parent base -> world; type fixed -> floating

File: data/laikago/urdf/laikago.urdf (robot description, URDF)
Before this commit: robot laikago_description, 13 links, 12 joints
Links:
- added link world
Joints:
- added joint floating_base: type floating, parent world, child trunk, origin xyz=0 0 0 rpy=0 0 0

Commit message: add go1

File: data/aliengo/urdf/aliengo.urdf (robot description, URDF)
Before this commit: robot aliengo_description, 19 links, 18 joints
Joints:
- removed joint 
- added joint floating_base: type floating, parent world, child trunk, origin xyz=0 0 0 rpy=0 0 0

File: data/laikago/urdf/laikago.urdf (robot description, URDF)
Before this commit: robot laikago_description, 14 links, 13 joints
Joints:
- removed joint 
- added joint floating_base: type floating, parent world, child trunk, origin xyz=0 0 0 rpy=0 0 0
